Commit message: feat: finaliza Prática 02 com xacro, gazebo_ros2_control e diff_drive

File: model_description/urdf/vasco_robot.urdf (robot description, URDF)
Before this commit: robot vasco_robot, 5 links, 4 joints
Links:
- added link cross_h; visual box size=0.08 0.02 0.01
- added link cross_v; visual box size=0.02 0.08 0.01
- added link white_stripe; visual box size=0.41 0.04 0.102
- link base_link: geometry collision box size=0.4 0.2 0.1; visual box size=0.4 0.2 0.1
Joints:
- added joint cross_h_joint: type fixed, parent base_link, child cross_h, origin xyz=0.08 0.05 0.055 rpy=0 0 0
- added joint cross_v_joint: type fixed, parent base_link, child cross_v, origin xyz=0.08 0.05 0.055 rpy=0 0 0
- added joint stripe_joint: type fixed, parent base_link, child white_stripe, origin xyz=0 0 0 rpy=0 0 0
