Commit message: pratica_03 finalizada

File: pratica_03/urdf/vasco_robot.urdf (robot description, URDF)
Before this commit: robot vasco_robot, 8 links, 7 joints
Links:
- link base_link: mass 5.0 -> 1.0
- link caster_wheel: mass 0.5 -> 0.25
- link left_wheel: mass 1.0 -> 0.5
- link right_wheel: mass 1.0 -> 0.5
Joints:
- joint left_wheel_joint: origin xyz=0.1 0.13 0 rpy=0 0 0 -> xyz=0.0 0.13 0 rpy=0 0 0
- joint right_wheel_joint: origin xyz=0.1 -0.13 0 rpy=0 0 0 -> xyz=0.0 -0.13 0 rpy=0 0 0
