Commit message: pratica_04 correcoes

File: pratica_04/urdf/vasco_robot.urdf (robot description, URDF)
Before this commit: robot vasco_robot, 13 links, 12 joints
Links:
- removed link caster_wheel_front
- removed link caster_wheel_rear
- added link caster_wheel, mass 0.25; collision sphere radius=0.05; visual sphere radius=0.05
- link base_link: mass 5.0 -> 1.0
- link left_wheel: mass 1.0 -> 0.5
- link right_wheel: mass 1.0 -> 0.5
Joints:
- removed joint caster_front_joint
- removed joint caster_rear_joint
- added joint caster_joint: type fixed, parent base_link, child caster_wheel, origin xyz=-0.15 0 -0.05 rpy=0 0 0
- joint left_wheel_joint: limit effort=1.5 velocity=10.0 -> (none); origin xyz=0 0.13 0 rpy=0 0 0 -> xyz=0.0 0.13 0 rpy=0 0 0
- joint right_wheel_joint: limit effort=1.5 velocity=10.0 -> (none); origin xyz=0 -0.13 0 rpy=0 0 0 -> xyz=0.0 -0.13 0 rpy=0 0 0
